Commit message: feat: checkpoint 2 — dual drive modes, active camera, ackermann fix
- URDF: added active 30 FPS camera sensor (libgazebo_ros_camera.so) on
  camera_link with proper optical frame (REP-103 camera_optical_link).
  Topics: /camera/image_raw, /camera/camera_info.

- URDF: dual drive mode xacro (drive_mode:=diff|ackermann).
  Diff mode: 4WD skid-steer via libgazebo_ros_diff_drive.so (num_wheel_pairs=2).
  Ackermann mode: steered front wheels (steer revolute + wheel continuous)
  driven via libgazebo_ros_ackermann_drive.so with stable PID tuning.

- Ackermann stability fix (three changes together):
  1. update_rate 100→500 Hz: keeps plugin timestep below closed-loop τ_cl
     (I/(D_mech+P) ≈ 5.5 ms); at 100 Hz the sampled controller was unstable.
  2. Wheel joint damping 0.05→0.005: widens stable P-gain range.
  3. PID: P=0.05, I=0.5, D=0 — D=0 avoids first-call derivative spike;
     I eliminates steady-state friction error. Steer: P=2.0, D=0.

- Launch: added drive_mode arg, pause/unpause after spawn (prevents NaN from
  GetVelocity(0) returning uninitialized value on first physics step),
  RViz2 camera display.

- CLAUDE.md: updated to CP2, documented ackermann stability root cause.

Co-Authored-By: Claude Sonnet 4.6 <noreply@anthropic.com>

File: src/robot_sim/urdf/limo_sim.urdf.xacro (robot description, xacro)
@@ -2,23 +2,36 @@
 <robot name="limo_sim" xmlns:xacro="http://ros.org/wiki/xacro">
   <!-- ================================================================
-       MATERIALS (used by RViz2)
-  ================================================================ -->
-  <material name="chassis_grey">
-    <color rgba="0.5 0.5 0.5 1.0"/>
-  </material>
-  <material name="wheel_black">
-    <color rgba="0.1 0.1 0.1 1.0"/>
-  </material>
-  <material name="caster_white">
-    <color rgba="0.9 0.9 0.9 1.0"/>
-  </material>
-  <material name="camera_blue">
-    <color rgba="0.0 0.4 0.8 1.0"/>
-  </material>
-  <material name="lidar_dark">
-    <color rgba="0.2 0.2 0.2 1.0"/>
-  </material>
-  <!-- ================================================================
-       BASE FOOTPRINT — root link, sits on ground plane
+       DRIVE MODE — 'diff' (4WD skid steer) or 'ackermann' (front-steer)
+       Pass via:  xacro limo_sim.urdf.xacro drive_mode:=ackermann
+  ================================================================ -->
+  <xacro:arg name="drive_mode" default="diff"/>
+  <xacro:property name="DRIVE_MODE" value="$(arg drive_mode)"/>
+  <!-- ================================================================
+       GEOMETRY CONSTANTS — LIMO Pro proportions (slightly stylized)
+  ================================================================ -->
+  <xacro:property name="WHEEL_RADIUS"   value="0.05"/>
+  <xacro:property name="WHEEL_WIDTH"    value="0.045"/>
+  <xacro:property name="WHEEL_MASS"     value="0.2"/>
+  <xacro:property name="WHEELBASE_HALF" value="0.10"/>   <!-- ±x distance from center -->
+  <xacro:property name="TRACK_HALF"     value="0.085"/>  <!-- ±y distance from center -->
+  <xacro:property name="BASE_Z"         value="0.075"/>  <!-- base_link height above ground -->
+  <xacro:property name="WHEEL_Z_OFFSET" value="-0.025"/> <!-- wheel center relative to base_link -->
+  <xacro:property name="CHASSIS_X"      value="0.32"/>
+  <xacro:property name="CHASSIS_Y"      value="0.22"/>
+  <xacro:property name="CHASSIS_Z"      value="0.06"/>
+  <xacro:property name="HOOD_X"         value="0.22"/>
+  <xacro:property name="HOOD_Y"         value="0.20"/>
+  <xacro:property name="HOOD_Z"         value="0.07"/>
+  <!-- ================================================================
+       MATERIALS (RViz2)
+  ================================================================ -->
+  <material name="limo_white"><color rgba="0.92 0.92 0.92 1.0"/></material>
+  <material name="limo_black"><color rgba="0.10 0.10 0.10 1.0"/></material>
+  <material name="limo_dark_grey"><color rgba="0.20 0.20 0.22 1.0"/></material>
+  <material name="limo_green"><color rgba="0.10 0.85 0.30 1.0"/></material>
+  <material name="wheel_black"><color rgba="0.05 0.05 0.05 1.0"/></material>
+  <material name="camera_lens"><color rgba="0.05 0.05 0.10 1.0"/></material>
+  <!-- ================================================================
+       ROOT FRAMES
   ================================================================ -->
   <link name="base_footprint"/>
@@ -26,267 +39,356 @@
     <parent link="base_footprint"/>
     <child link="base_link"/>
-    <origin xyz="0.0 0.0 0.1" rpy="0 0 0"/>
+    <origin xyz="0 0 ${BASE_Z}" rpy="0 0 0"/>
   </joint>
   <!-- ================================================================
-       BASE LINK — chassis
-       Box: 0.4m(x) x 0.3m(y) x 0.12m(z), mass=4kg
-       Inertia (solid box):
-         ixx = m/12*(y^2+z^2) = 4/12*(0.09+0.0144) = 0.0348
-         iyy = m/12*(x^2+z^2) = 4/12*(0.16+0.0144) = 0.0581
-         izz = m/12*(x^2+y^2) = 4/12*(0.16+0.09)   = 0.0833
+       BASE LINK — composite chassis: white lower deck + black upper hood
+                   + tilted dark front cowl + side accents + antennas.
+       Inertia approximated as solid box of CHASSIS dims + hood mass.
+       Body mass ≈ 4.0 kg.
   ================================================================ -->
   <link name="base_link">
+    <!-- Lower white deck -->
     <visual>
       <origin xyz="0 0 0" rpy="0 0 0"/>
-      <geometry><box size="0.4 0.3 0.12"/></geometry>
-      <material name="chassis_grey"/>
+      <geometry><box size="${CHASSIS_X} ${CHASSIS_Y} ${CHASSIS_Z}"/></geometry>
+      <material name="limo_white"/>
+    </visual>
+    <!-- Upper black hood -->
+    <visual>
+      <origin xyz="-0.02 0 ${CHASSIS_Z/2 + HOOD_Z/2}" rpy="0 0 0"/>
+      <geometry><box size="${HOOD_X} ${HOOD_Y} ${HOOD_Z}"/></geometry>
+      <material name="limo_black"/>
+    </visual>
+    <!-- Tilted front cowl (tablet-style screen) -->
+    <visual>
+      <origin xyz="0.10 0 ${CHASSIS_Z/2 + 0.045}" rpy="0 -0.45 0"/>
+      <geometry><box size="0.06 0.18 0.09"/></geometry>
+      <material name="limo_dark_grey"/>
+    </visual>
+    <!-- Left green LED accent strip -->
+    <visual>
+      <origin xyz="0.06 ${CHASSIS_Y/2 + 0.001} 0.005" rpy="0 0 0"/>
+      <geometry><box size="0.03 0.005 0.015"/></geometry>
+      <material name="limo_green"/>
+    </visual>
+    <!-- Right green LED accent strip -->
+    <visual>
+      <origin xyz="0.06 ${-CHASSIS_Y/2 - 0.001} 0.005" rpy="0 0 0"/>
+      <geometry><box size="0.03 0.005 0.015"/></geometry>
+      <material name="limo_green"/>
+    </visual>
+    <!-- Left antenna -->
+    <visual>
+      <origin xyz="-0.07 0.05 ${CHASSIS_Z/2 + HOOD_Z + 0.03}" rpy="0 0 0"/>
+      <geometry><cylinder radius="0.0035" length="0.06"/></geometry>
+      <material name="limo_black"/>
+    </visual>
+    <!-- Right antenna -->
+    <visual>
+      <origin xyz="-0.07 -0.05 ${CHASSIS_Z/2 + HOOD_Z + 0.03}" rpy="0 0 0"/>
+      <geometry><cylinder radius="0.0035" length="0.06"/></geometry>
+      <material name="limo_black"/>
+    </visual>
+    <!-- Collision: single bounding box covering deck + hood -->
+    <collision>
+      <origin xyz="0 0 0.04" rpy="0 0 0"/>
+      <geometry><box size="${CHASSIS_X} ${CHASSIS_Y} 0.14"/></geometry>
+    </collision>
+    <inertial>
+      <origin xyz="0 0 0.03" rpy="0 0 0"/>
+      <mass value="4.0"/>
+      <!-- Solid box (0.32 x 0.22 x 0.14): ixx=m/12*(y²+z²), iyy=m/12*(x²+z²), izz=m/12*(x²+y²) -->
+      <inertia ixx="0.022667" ixy="0" ixz="0"
+               iyy="0.040667" iyz="0"
+               izz="0.050267"/>
+    </inertial>
+  </link>
+  <!-- ================================================================
+       WHEEL MACRO — fixed-position spinning wheel
+       Used for: all 4 wheels in 'diff' mode, rear 2 wheels in 'ackermann'.
+       Joint spins around Y axis directly (no joint-origin rotation).
+       Visual/collision rotate cylinder so its long axis aligns with Y.
+  ================================================================ -->
+  <xacro:macro name="fixed_wheel" params="prefix x y">
+    <joint name="${prefix}_wheel_joint" type="continuous">
+      <parent link="base_link"/>
+      <child  link="${prefix}_wheel_link"/>
+      <origin xyz="${x} ${y} ${WHEEL_Z_OFFSET}" rpy="0 0 0"/>
+      <axis xyz="0 1 0"/>
+      <dynamics damping="0.005" friction="0.005"/>
+    </joint>
+    <link name="${prefix}_wheel_link">
+      <visual>
+        <origin xyz="0 0 0" rpy="1.5707963 0 0"/>
+        <geometry><cylinder radius="${WHEEL_RADIUS}" length="${WHEEL_WIDTH}"/></geometry>
+        <material name="wheel_black"/>
+      </visual>
+      <collision>
+        <origin xyz="0 0 0" rpy="1.5707963 0 0"/>
+        <geometry><cylinder radius="${WHEEL_RADIUS}" length="${WHEEL_WIDTH}"/></geometry>
+      </collision>
+      <inertial>
+        <origin xyz="0 0 0" rpy="0 0 0"/>
+        <mass value="${WHEEL_MASS}"/>
+        <!-- Cylinder rotated to spin about Y: principal axis is now Y.
+             ixx=izz=m/12*(3r²+l²) = 0.000159
+             iyy=m/2*r²            = 0.000250 -->
+        <inertia ixx="0.000159" ixy="0" ixz="0"
+                 iyy="0.000250" iyz="0"
+                 izz="0.000159"/>
+      </inertial>
+    </link>
+    <gazebo reference="${prefix}_wheel_link">
+      <material>Gazebo/FlatBlack</material>
+      <mu1>1.2</mu1>
+      <mu2>1.0</mu2>
+      <kp>1000000.0</kp>
+      <kd>100.0</kd>
+      <minDepth>0.001</minDepth>
+      <maxVel>0.5</maxVel>
+      <fdir1>1 0 0</fdir1>
+    </gazebo>
+  </xacro:macro>
+  <!-- ================================================================
+       STEERED WHEEL MACRO — 2-DOF: steer revolute + spin continuous.
+       Used only for front 2 wheels in 'ackermann' mode.
+  ================================================================ -->
+  <xacro:macro name="steered_wheel" params="prefix x y">
+    <!-- Steering link: tiny massless dummy that pivots about Z -->
+    <joint name="${prefix}_steer_joint" type="revolute">
+      <parent link="base_link"/>
+      <child  link="${prefix}_steer_link"/>
+      <origin xyz="${x} ${y} ${WHEEL_Z_OFFSET}" rpy="0 0 0"/>
+      <axis xyz="0 0 1"/>
+      <limit lower="-0.6" upper="0.6" effort="50" velocity="3.0"/>
+      <dynamics damping="0.3" friction="0.02"/>
+    </joint>
+    <link name="${prefix}_steer_link">
+      <inertial>
+        <origin xyz="0 0 0" rpy="0 0 0"/>
+        <mass value="0.2"/>
+        <inertia ixx="0.0002" ixy="0" ixz="0"
+                 iyy="0.0002" iyz="0"
+                 izz="0.0002"/>
+      </inertial>
+    </link>
+    <!-- Wheel link: spins about Y axis directly (no joint-origin rotation) -->
+    <joint name="${prefix}_wheel_joint" type="continuous">
+      <parent link="${prefix}_steer_link"/>
+      <child  link="${prefix}_wheel_link"/>
+      <origin xyz="0 0 0" rpy="0 0 0"/>
+      <axis xyz="0 1 0"/>
+      <dynamics damping="0.005" friction="0.005"/>
+    </joint>
+    <link name="${prefix}_wheel_link">
+      <visual>
+        <origin xyz="0 0 0" rpy="1.5707963 0 0"/>
+        <geometry><cylinder radius="${WHEEL_RADIUS}" length="${WHEEL_WIDTH}"/></geometry>
+        <material name="wheel_black"/>
+      </visual>
+      <collision>
+        <origin xyz="0 0 0" rpy="1.5707963 0 0"/>
+        <geometry><cylinder radius="${WHEEL_RADIUS}" length="${WHEEL_WIDTH}"/></geometry>
+      </collision>
+      <inertial>
+        <origin xyz="0 0 0" rpy="0 0 0"/>
+        <mass value="${WHEEL_MASS}"/>
+        <!-- Cylinder spins about Y: iyy=m/2*r², ixx=izz=m/12*(3r²+l²) -->
+        <inertia ixx="0.000159" ixy="0" ixz="0"
+                 iyy="0.000250" iyz="0"
+                 izz="0.000159"/>
+      </inertial>
+    </link>
+    <gazebo reference="${prefix}_wheel_link">
+      <material>Gazebo/FlatBlack</material>
+      <mu1>1.2</mu1>
+      <mu2>1.0</mu2>
+      <kp>1000000.0</kp>
+      <kd>100.0</kd>
+      <minDepth>0.001</minDepth>
+      <maxVel>0.5</maxVel>
+      <fdir1>1 0 0</fdir1>
+    </gazebo>
+  </xacro:macro>
+  <!-- ================================================================
+       FRONT WHEELS — steered in ackermann, fixed in diff
+  ================================================================ -->
+  <xacro:if value="${DRIVE_MODE == 'ackermann'}">
+    <xacro:steered_wheel prefix="front_left"  x="${WHEELBASE_HALF}" y="${TRACK_HALF}"/>
+    <xacro:steered_wheel prefix="front_right" x="${WHEELBASE_HALF}" y="${-TRACK_HALF}"/>
+  </xacro:if>
+  <xacro:if value="${DRIVE_MODE == 'diff'}">
+    <xacro:fixed_wheel prefix="front_left"  x="${WHEELBASE_HALF}" y="${TRACK_HALF}"/>
+    <xacro:fixed_wheel prefix="front_right" x="${WHEELBASE_HALF}" y="${-TRACK_HALF}"/>
+  </xacro:if>
+  <!-- REAR WHEELS — always fixed-position spinning -->
+  <xacro:fixed_wheel prefix="rear_left"  x="${-WHEELBASE_HALF}" y="${TRACK_HALF}"/>
+  <xacro:fixed_wheel prefix="rear_right" x="${-WHEELBASE_HALF}" y="${-TRACK_HALF}"/>
+  <!-- ================================================================
+       CAMERA — small dark protrusion at top of front cowl.
+       camera_link is the URDF/visual frame (REP-103 ENU: x-forward).
+       camera_optical_link is the optical frame used by image_raw
+       (REP-103: x-right, y-down, z-forward).
+  ================================================================ -->
+  <joint name="camera_joint" type="fixed">
+    <parent link="base_link"/>
+    <child  link="camera_link"/>
+    <origin xyz="0.135 0 0.10" rpy="0 0 0"/>
+  </joint>
+  <link name="camera_link">
+    <visual>
+      <origin xyz="0 0 0" rpy="0 0 0"/>
+      <geometry><box size="0.02 0.06 0.025"/></geometry>
+      <material name="camera_lens"/>
     </visual>
     <collision>
       <origin xyz="0 0 0" rpy="0 0 0"/>
-      <geometry><box size="0.4 0.3 0.12"/></geometry>
+      <geometry><box size="0.02 0.06 0.025"/></geometry>
     </collision>
     <inertial>
       <origin xyz="0 0 0" rpy="0 0 0"/>
-      <mass value="4.0"/>
-      <inertia ixx="0.034800" ixy="0" ixz="0"
-               iyy="0.058133" iyz="0"
-               izz="0.083333"/>
+      <mass value="0.03"/>
+      <inertia ixx="1e-5" ixy="0" ixz="0"
+               iyy="1e-5" iyz="0"
+               izz="1e-5"/>
     </inertial>
   </link>
-  <!-- ================================================================
-       LEFT DRIVE WHEEL
-       origin y=+0.085 (half of 0.17m track width)
-       origin z=-0.055 (wheel_radius 0.045 - base_link_z_offset 0.1)
-       rpy=-pi/2 rotates cylinder so its long axis aligns with world Y.
-       axis="0 0 1" then means spin around local Z = world Y.
-  ================================================================ -->
-  <joint name="left_wheel_joint" type="continuous">
-    <parent link="base_link"/>
-    <child link="left_wheel_link"/>
-    <origin xyz="0.0 0.085 -0.055" rpy="-1.5707963 0 0"/>
-    <axis xyz="0 0 1"/>
+  <joint name="camera_optical_joint" type="fixed">
+    <parent link="camera_link"/>
+    <child  link="camera_optical_link"/>
+    <!-- Rotate URDF frame (x-fwd, y-left, z-up) → optical (x-right, y-down, z-fwd) -->
+    <origin xyz="0 0 0" rpy="-1.5707963 0 -1.5707963"/>
   </joint>
-  <link name="left_wheel_link">
-    <visual>
-      <origin xyz="0 0 0" rpy="0 0 0"/>
-      <geometry><cylinder radius="0.045" length="0.04"/></geometry>
-      <material name="wheel_black"/>
-    </visual>
-    <collision>
-      <origin xyz="0 0 0" rpy="0 0 0"/>
-      <geometry><cylinder radius="0.045" length="0.04"/></geometry>
-    </collision>
-    <inertial>
-      <origin xyz="0 0 0" rpy="0 0 0"/>
-      <mass value="0.15"/>
-      <!-- Cylinder: ixx=iyy=m/12*(3r^2+l^2), izz=m/2*r^2 -->
-      <inertia ixx="0.000096" ixy="0" ixz="0"
-               iyy="0.000096" iyz="0"
-               izz="0.000152"/>
-    </inertial>
-  </link>
-  <!-- ================================================================
-       RIGHT DRIVE WHEEL
-  ================================================================ -->
-  <joint name="right_wheel_joint" type="continuous">
-    <parent link="base_link"/>
-    <child link="right_wheel_link"/>
-    <origin xyz="0.0 -0.085 -0.055" rpy="-1.5707963 0 0"/>
-    <axis xyz="0 0 1"/>
-  </joint>
-  <link name="right_wheel_link">
-    <visual>
-      <origin xyz="0 0 0" rpy="0 0 0"/>
-      <geometry><cylinder radius="0.045" length="0.04"/></geometry>
-      <material name="wheel_black"/>
-    </visual>
-    <collision>
-      <origin xyz="0 0 0" rpy="0 0 0"/>
-      <geometry><cylinder radius="0.045" length="0.04"/></geometry>
-    </collision>
-    <inertial>
-      <origin xyz="0 0 0" rpy="0 0 0"/>
-      <mass value="0.15"/>
-      <inertia ixx="0.000096" ixy="0" ixz="0"
-               iyy="0.000096" iyz="0"
-               izz="0.000152"/>
-    </inertial>
-  </link>
-  <!-- ================================================================
-       FRONT CASTER WHEELS (fixed, frictionless spheres)
-       z = -(base_link_z_offset - caster_radius) = -(0.1 - 0.025) = -0.075
-  ================================================================ -->
-  <joint name="front_caster_left_joint" type="fixed">
-    <parent link="base_link"/>
-    <child link="front_caster_left_link"/>
-    <origin xyz="0.15 0.06 -0.075" rpy="0 0 0"/>
-  </joint>
-  <link name="front_caster_left_link">
-    <visual>
-      <origin xyz="0 0 0" rpy="0 0 0"/>
-      <geometry><sphere radius="0.025"/></geometry>
-      <material name="caster_white"/>
-    </visual>
-    <collision>
-      <origin xyz="0 0 0" rpy="0 0 0"/>
-      <geometry><sphere radius="0.025"/></geometry>
-    </collision>
-    <inertial>
-      <origin xyz="0 0 0" rpy="0 0 0"/>
-      <mass value="0.05"/>
-      <!-- Sphere: i = 2/5*m*r^2 -->
-      <inertia ixx="0.0000125" ixy="0" ixz="0"
-               iyy="0.0000125" iyz="0"
-               izz="0.0000125"/>
-    </inertial>
-  </link>
-  <joint name="front_caster_right_joint" type="fixed">
-    <parent link="base_link"/>
-    <child link="front_caster_right_link"/>
-    <origin xyz="0.15 -0.06 -0.075" rpy="0 0 0"/>
-  </joint>
-  <link name="front_caster_right_link">
-    <visual>
-      <origin xyz="0 0 0" rpy="0 0 0"/>
-      <geometry><sphere radius="0.025"/></geometry>
-      <material name="caster_white"/>
-    </visual>
-    <collision>
-      <origin xyz="0 0 0" rpy="0 0 0"/>
-      <geometry><sphere radius="0.025"/></geometry>
-    </collision>
-    <inertial>
-      <origin xyz="0 0 0" rpy="0 0 0"/>
-      <mass value="0.05"/>
-      <inertia ixx="0.0000125" ixy="0" ixz="0"
-               iyy="0.0000125" iyz="0"
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